File: KiCAD/Mimosa/Mimosa.kicad_sch (KiCad schematic)
At the start: 0 parts

Commit message: Updating
Parts:
- added C1, C7: 1uF, Capacitor_SMD:C_0603_1608Metric, symbol Device:C
- added C2: 4.7uF, Capacitor_SMD:C_0603_1608Metric, symbol Device:C
- added C3, C4, C5, C8, C9: 100nF, Capacitor_SMD:C_0603_1608Metric, symbol Device:C
- added C6: 22uF, Capacitor_SMD:C_0603_1608Metric, symbol Device:C
- added R1: R, Resistor_SMD:R_0805_2012Metric, symbol Device:R
- added U1: LDL1117S33R, lcsc_footprints:C435835_SOT-223-4_L6_5-W3_5-P2_30-LS7_0-BR, symbol lcsc_imported:LDL1117S33R
- added U2: MSM381ACP003_C51928212, lcsc_footprints:C51928212_MIC-SMD_4P-L2_8-W1_9-TR_MSM381ACP003, symbol lcsc_imported:MSM381ACP003_C51928212
- added U3: SGM5353-16XS8G/TR, lcsc_footprints:C5152099_SOIC-8_L4_9-W3_9-P1_27-LS6_0-BL, symbol lcsc_imported:SGM5353-16XS8G/TR
- added U4: AD4680BCPZ-RL7, lcsc_footprints:C5548270_LFCSP-16_L3_0-W3_0-P0_50-TL-EP1_1, symbol lcsc_imported:AD4680BCPZ-RL7
- added U5: ESP32-S3-WROOM-1-N8, lcsc_footprints:C2913198_WIFIM-SMD_ESP32-S3-WROOM-1-N8, symbol lcsc_imported:ESP32-S3-WROOM-1-N8
- added U6: D3V3XA4B10LP, Package_DFN_QFN:Diodes_UDFN-10_1x2.5mm_P0.5mm, symbol Power_Protection:D3V3XA4B10LP
- added USB1: MICRO5.9MMUSB, lcsc_footprints:C393940_MICRO-USB-SMD_5P-P0_65-H-F_MICRO5_9MMUSB, symbol lcsc_imported:MICRO5_9MMUSB
Connections:
- new net: R1.1, U5.3 (EN)
- new net 3.3V: C2.1, C4.1, C5.2, C6.2, R1.2, U1.2 (VOUT), U1.4 (VOUT), U5.2 (3V3)
- new net D+: U6.5, U6.6 (NC), USB1.3 (D+)
- new net D-: U6.4, U6.7 (NC), USB1.2 (D-)
- new net GND: C1.2, C2.2, C3.2, C4.2, C5.1, C6.1, U1.1 (GND), U5.1 (GND), U5.40 (GND), U5.41 (EP), U6.3 (VSS), U6.8 (VSS), USB1.5 (GND), USB1.6
- new net Vbus: U6.1, U6.10 (NC), USB1.1 (VBUS)
- new net Vin: C1.1, C3.1, U1.3 (VIN)
- no-connect marks 0 -> 3
Other:
- note added: "Regulador 3.3V"
- note added: "USB"

Commit message: Updating 2
Parts:
- added J1: Conn_01x02_Pin, Connector_Molex:Molex_KK-396_A-41791-0002_1x02_P3.96mm_Vertical, symbol Connector:Conn_01x02_Pin
- added U7: NAU8810YG, lcsc_footprints:C2613464_QFN-20_L4_0-W4_0-P0_5-EP2_0, symbol lcsc_imported:NAU8810YG
- added U8: BL4056C-42ES, lcsc_footprints:C918909_ESOP-8_L4_9-W3_9-P1_27-LS6_0-BL-EP, symbol lcsc_imported:BL4056C-42ES
